Commit message: Add files via upload

File: mi_TFG/urdf/dron_plugins.xacro (robot description, xacro)
@@ -16,4 +16,6 @@
     <xacro:arg name="fisico_motores_masa" default="0.05"/>
     <xacro:arg name="fisico_motores_matriz_inercia" default="1e-5 1e-5 1e-5 0 0 0"/>
+    <xacro:arg name="actuadores_conversor_fuerza2torque" default="0.02"/>
+    <xacro:arg name="sensores_ground_truth_publish_rate" default="50.0"/>
     <!-- Se pasa a propiedad para poder hacer cálculos con ella -->
     <xacro:property name="fisico_cuerpo_dim" value="$(arg fisico_cuerpo_dim)"/>
@@ -31,4 +33,6 @@
     <xacro:property name="fisico_motores_masa" value="$(arg fisico_motores_masa)"/>
     <xacro:property name="fisico_motores_matriz_inercia" value="$(arg fisico_motores_matriz_inercia)"/>
+    <xacro:property name="actuadores_conversor_fuerza2torque" value="$(arg actuadores_conversor_fuerza2torque)"/>
+    <xacro:property name="sensores_ground_truth_publish_rate" value="$(arg sensores_ground_truth_publish_rate)"/>
     <!-- Materiales -->
     <material name="White"><color rgba="1.0 1.0 1.0 1.0"/></material>
@@ -119,11 +123,27 @@
     <!-- MACRO 4 Brazos -->
     <xacro:if value="${fisico_brazos_numero == 4}">
+        <!-- Crear Brazos -->
         <xacro:brazo_total name="arriba_izquierda" yaw="${fisico_brazos_grados/180*pi}"/>
         <xacro:brazo_total name="abajo_izquierda" yaw="${pi - fisico_brazos_grados/180*pi}"/>
         <xacro:brazo_total name="abajo_derecha" yaw="${pi + fisico_brazos_grados/180*pi}"/>
         <xacro:brazo_total name="arriba_derecha" yaw="${- fisico_brazos_grados/180*pi}"/>
+        <!-- Plugin Motores -->
+        <gazebo>
+            <plugin name="plugin_actuar_motores" filename="libplugin_actuar_motores.so">
+                <motor1>arriba_izquierda_motor</motor1>
+                <topic1>motor/arr_iz</topic1>
+                <motor2>abajo_izquierda_motor</motor2>
+                <topic2>motor/ab_iz</topic2>
+                <motor3>abajo_derecha_motor</motor3>
+                <topic3>motor/ab_der</topic3>
+                <motor4>arriba_derecha_motor</motor4>
+                <topic4>motor/arr_der</topic4>
+                <fuerza2torque>${actuadores_conversor_fuerza2torque}</fuerza2torque>
+            </plugin>
+        </gazebo>
     </xacro:if>
     <!-- MACRO 6 Brazos -->
     <xacro:if value="${fisico_brazos_numero == 6}">
+        <!-- Crear Brazos -->
         <xacro:brazo_total name="arriba_izquierda" yaw="${fisico_brazos_grados/180*pi}"/>
         <xacro:brazo_total name="izquierda" yaw="${pi/2}"/>
@@ -132,7 +152,26 @@
         <xacro:brazo_total name="derecha" yaw="${-pi/2}"/>
         <xacro:brazo_total name="arriba_derecha" yaw="${- fisico_brazos_grados/180*pi}"/>
+        <!-- Plugin Motores -->
+        <gazebo>
+            <plugin name="plugin_actuar_motores" filename="libplugin_actuar_motores.so">
+                <motor1>arriba_izquierda_motor</motor1>
+                <topic1>motor/arr_iz</topic1>
+                <motor2>izquierda_motor</motor2>
+                <topic2>motor/iz</topic2>
+                <motor3>abajo_izquierda_motor</motor3>
+                <topic3>motor/ab_iz</topic3>
+                <motor4>abajo_derecha_motor</motor4>
+                <topic4>motor/ab_der</topic4>
+                <motor5>derecha_motor</motor5>
+                <topic5>motor/der</topic5>
+                <motor6>arriba_derecha_motor</motor6>
+                <topic6>motor/arr_der</topic6>
+                <fuerza2torque>${actuadores_conversor_fuerza2torque}</fuerza2torque>
+            </plugin>
+        </gazebo>
     </xacro:if>
     <!-- MACRO 8 Brazos -->
     <xacro:if value="${fisico_brazos_numero == 8}">
+        <!-- Crear Brazos -->
         <xacro:brazo_total name="arriba" yaw="0"/>
         <xacro:brazo_total name="arriba_izquierda" yaw="${fisico_brazos_grados/180*pi}"/>
@@ -143,4 +182,38 @@
         <xacro:brazo_total name="derecha" yaw="${-pi/2}"/>
         <xacro:brazo_total name="arriba_derecha" yaw="${- fisico_brazos_grados/180*pi}"/>
+        <!-- Plugin Motores -->
+        <gazebo>
+            <plugin name="plugin_actuar_motores" filename="libplugin_actuar_motores.so">
+                <motor1>arriba_motor</motor1>
+                <topic1>motor/arr</topic1>
+                <motor2>arriba_izquierda_motor</motor2>
+                <topic2>motor/arr_iz</topic2>
+                <motor3>izquierda_motor</motor3>
+                <topic3>motor/iz</topic3>
+                <motor4>abajo_izquierda_motor</motor4>
+                <topic4>motor/ab_iz</topic4>
+                <motor5>abajo_motor</motor5>
+                <topic5>motor/ab</topic5>
+                <motor6>abajo_derecha_motor</motor6>
+                <topic6>motor/ab_der</topic6>
+                <motor7>derecha_motor</motor7>
+                <topic7>motor/der</topic7>
+                <motor8>arriba_derecha_motor</motor8>
+                <topic8>motor/arr_der</topic8>
+                <fuerza2torque>${actuadores_conversor_fuerza2torque}</fuerza2torque>
+            </plugin>
+        </gazebo>
     </xacro:if>
+    <!-- Plugin GroundTruth -->
+    <gazebo>
+        <plugin name="plugin_sensor_groundtrurh" filename="libplugin_sensor_groundtrurh.so">
+            <link_name>cuerpo</link_name>
+            <topic_pose>sensor/GT/pose</topic_pose>
+            <topic_vel>sensor/GT/vel</topic_vel>
+            <topic_acc>sensor/GT/acc</topic_acc>
+            <publish_rate>${sensores_ground_truth_publish_rate}</publish_rate>
+            <frame_id>world</frame_id>
+            <frame_propio>false</frame_propio>
+        </plugin>
+    </gazebo>
 </robot>

Commit message: Add files via upload

File: mi_TFG/urdf/dron_plugins.xacro (robot description, xacro)
@@ -16,6 +16,13 @@
     <xacro:arg name="fisico_motores_masa" default="0.05"/>
     <xacro:arg name="fisico_motores_matriz_inercia" default="1e-5 1e-5 1e-5 0 0 0"/>
+    <xacro:arg name="fisico_camara_dim" default="0.005 0.01 0.01"/>
+    <xacro:arg name="fisico_camara_color" default="Yellow"/>
+    <xacro:arg name="fisico_camara_masa" default="0.01"/>
+    <xacro:arg name="fisico_camara_matriz_inercia" default="1e-6 1e-6 1e-6 0 0 0"/>
     <xacro:arg name="actuadores_conversor_fuerza2torque" default="0.02"/>
     <xacro:arg name="sensores_ground_truth_publish_rate" default="50.0"/>
+    <xacro:arg name="sensores_camara_porcentaje_estereo" default= "0.3"/>
+    <xacro:arg name="sensores_camara_publish_rate" default= "30.0"/>
+    <xacro:arg name="sensores_camara_mostrar_gazebo" default= "false"/>
     <!-- Se pasa a propiedad para poder hacer cálculos con ella -->
     <xacro:property name="fisico_cuerpo_dim" value="$(arg fisico_cuerpo_dim)"/>
@@ -33,10 +40,20 @@
     <xacro:property name="fisico_motores_masa" value="$(arg fisico_motores_masa)"/>
     <xacro:property name="fisico_motores_matriz_inercia" value="$(arg fisico_motores_matriz_inercia)"/>
+    <xacro:property name="fisico_camara_dim" value="$(arg fisico_camara_dim)"/>
+    <xacro:property name="fisico_camara_color" value="$(arg fisico_camara_color)"/>
+    <xacro:property name="fisico_camara_masa" value="$(arg fisico_camara_masa)"/>
+    <xacro:property name="fisico_camara_matriz_inercia" value="$(arg fisico_camara_matriz_inercia)"/>
     <xacro:property name="actuadores_conversor_fuerza2torque" value="$(arg actuadores_conversor_fuerza2torque)"/>
     <xacro:property name="sensores_ground_truth_publish_rate" value="$(arg sensores_ground_truth_publish_rate)"/>
+    <xacro:property name="sensores_camara_porcentaje_estereo" value="$(arg sensores_camara_porcentaje_estereo)"/>
+    <xacro:property name="sensores_camara_publish_rate" value="$(arg sensores_camara_publish_rate)"/>
+    <xacro:property name="sensores_camara_mostrar_gazebo" value="$(arg sensores_camara_mostrar_gazebo)"/>
     <!-- Materiales -->
     <material name="White"><color rgba="1.0 1.0 1.0 1.0"/></material>
     <material name="Gray"><color rgba="0.5 0.5 0.5 1.0"/></material>
     <material name="Red"><color rgba="1.0 0.0 0.0 1.0"/></material>
+    <material name="Green"><color rgba="0.0 1.0 0.0 1.0"/></material>
+    <material name="Magenta"><color rgba="1.0 0.0 0.5 1.0"/></material>
+    <material name="Yellow"><color rgba="0.0 1.0 1.0 1.0"/></material>
     <!-- Cuerpo central -->
     <link name="cuerpo">
@@ -217,3 +234,81 @@
         </plugin>
     </gazebo>
+    <!-- MACRO Link Camara -->
+    <xacro:macro name="link_camara" params="name">
+        <link name="camara_${name}">
+            <visual>
+                <geometry><box size="${fisico_camara_dim}"/></geometry>
+                <material name="${fisico_camara_color}"/>
+            </visual>
+            <collision>
+                <geometry><box size="${fisico_camara_dim}"/></geometry>
+            </collision>
+            <inertial>
+                <mass value="${fisico_camara_masa}"/>
+                <inertia ixx="${fisico_camara_matriz_inercia.split()[0]}" iyy="${fisico_camara_matriz_inercia.split()[1]}" izz="${fisico_camara_matriz_inercia.split()[2]}" ixy="${fisico_camara_matriz_inercia.split()[3]}" ixz="${fisico_camara_matriz_inercia.split()[4]}" iyz="${fisico_camara_matriz_inercia.split()[5]}"/>
+            </inertial>
+        </link>
+        <gazebo reference="camara_${name}">
+            <material>Gazebo/${fisico_camara_color}</material>
+        </gazebo>
+        <gazebo reference="camara_${name}">
+            <sensor name="sensor/camera_${name}" type="camera">
+                <always_on>true</always_on>         <!-- Si "true": El tópico funciona aunque nadie se suscriba -->
+                <update_rate>${sensores_camara_publish_rate}</update_rate>       <!-- FPS -->
+                <visualize>${sensores_camara_mostrar_gazebo}</visualize>         <!-- Muestra lo que ve en gazebo -->
+                <pose>0 0 0 0 0 0</pose>            <!-- Pose respecto al link -->
+                <camera>
+                    <horizontal_fov>1.3962634</horizontal_fov>      <!-- Campo de visión: 80º aprox -->
+                    <image>
+                        <width>640</width>
+                        <height>480</height>
+                        <format>R8G8B8</format>
+                    </image>
+                    <clip>
+                        <near>0.05</near>       <!-- Distancia mínima a la que el sensor empieza a ver -->
+                        <far>50.0</far>         <!-- Distancia máxima a la que el sensor deja de ver -->
+                    </clip>
+                </camera>
+                <!-- SOLO Gazebo Classic -->
+                <plugin name="camera_controller_${name}" filename="libgazebo_ros_camera.so">
+                    <robotNamespace>/</robotNamespace>
+                    <cameraName>camara_${name}</cameraName>
+                    <imageTopicName>sensor/camara_${name}/image_raw</imageTopicName>
+                    <cameraInfoTopicName>sensor/camara_${name}/camera_info</cameraInfoTopicName>
+                    <frameName>camara_${name}</frameName>
+                </plugin>
+            </sensor>
+        </gazebo>
+    </xacro:macro>
+    <!-- MACRO Joint Cuerpo - Camara (mono)-->
+    <xacro:macro name="joint_camara_mono" params="name">
+        <xacro:property name="ox" value="${0.5 * float(fisico_cuerpo_dim.split()[0]) - 0.5 * float(fisico_camara_dim.split()[0])}"/>
+        <xacro:property name="oz" value="${0.5 * float(fisico_cuerpo_dim.split()[2]) + 0.5 * float(fisico_camara_dim.split()[2])}"/>
+        <joint name="joint_camara_${name}" type="fixed">
+            <parent link="cuerpo"/>
+            <child link="camara_${name}"/>
+            <origin xyz="${ox} 0 ${oz}" rpy="0 0 0"/>
+        </joint>
+    </xacro:macro>
+    <!-- MACRO Joint Cuerpo - Camara (estereo)-->
+    <xacro:macro name="joint_camara_estereo" params="name derecha">
+        <xacro:property name="ox" value="${0.5 * float(fisico_cuerpo_dim.split()[0]) - 0.5 * float(fisico_camara_dim.split()[0])}"/>
+        <xacro:property name="oz" value="${0.5 * float(fisico_cuerpo_dim.split()[2]) + 0.5 * float(fisico_camara_dim.split()[2])}"/>
+        <xacro:property name="oy" value="${(0.5 * float(fisico_cuerpo_dim.split()[1]) - 0.5 * float(fisico_camara_dim.split()[1]))*derecha*sensores_camara_porcentaje_estereo}"/>
+        <joint name="joint_camara_${name}" type="fixed">
+            <parent link="cuerpo"/>
+            <child link="camara_${name}"/>
+            <origin xyz="${ox} ${oy} ${oz}" rpy="0 0 0"/>
+        </joint>
+    </xacro:macro>
+    <xacro:if value="${sensores_camara_porcentaje_estereo == 0.0}">
+        <xacro:link_camara name="mono"/>
+        <xacro:joint_camara_mono name="mono"/>
+    </xacro:if>
+    <xacro:unless value="${sensores_camara_porcentaje_estereo == 0.0}">
+        <xacro:link_camara name="izq"/>
+        <xacro:joint_camara_estereo name="izq" derecha="-1.0"/>
+        <xacro:link_camara name="der"/>
+        <xacro:joint_camara_estereo name="der" derecha="1.0"/>
+    </xacro:unless>
 </robot>

Commit message: Add files via upload

File: mi_TFG/urdf/dron_plugins.xacro (robot description, xacro)
@@ -253,5 +253,5 @@
         </gazebo>
         <gazebo reference="camara_${name}">
-            <sensor name="sensor/camera_${name}" type="camera">
+            <sensor name="sensor/camara_${name}" type="camera">
                 <always_on>true</always_on>         <!-- Si "true": El tópico funciona aunque nadie se suscriba -->
                 <update_rate>${sensores_camara_publish_rate}</update_rate>       <!-- FPS -->
@@ -292,8 +292,8 @@
     </xacro:macro>
     <!-- MACRO Joint Cuerpo - Camara (estereo)-->
-    <xacro:macro name="joint_camara_estereo" params="name derecha">
+    <xacro:macro name="joint_camara_estereo" params="name izquierda">
         <xacro:property name="ox" value="${0.5 * float(fisico_cuerpo_dim.split()[0]) - 0.5 * float(fisico_camara_dim.split()[0])}"/>
         <xacro:property name="oz" value="${0.5 * float(fisico_cuerpo_dim.split()[2]) + 0.5 * float(fisico_camara_dim.split()[2])}"/>
-        <xacro:property name="oy" value="${(0.5 * float(fisico_cuerpo_dim.split()[1]) - 0.5 * float(fisico_camara_dim.split()[1]))*derecha*sensores_camara_porcentaje_estereo}"/>
+        <xacro:property name="oy" value="${(0.5 * float(fisico_cuerpo_dim.split()[1]) - 0.5 * float(fisico_camara_dim.split()[1]))*izquierda*sensores_camara_porcentaje_estereo}"/>
         <joint name="joint_camara_${name}" type="fixed">
             <parent link="cuerpo"/>
@@ -308,7 +308,7 @@
     <xacro:unless value="${sensores_camara_porcentaje_estereo == 0.0}">
         <xacro:link_camara name="izq"/>
-        <xacro:joint_camara_estereo name="izq" derecha="-1.0"/>
+        <xacro:joint_camara_estereo name="izq" izquierda="1.0"/>
         <xacro:link_camara name="der"/>
-        <xacro:joint_camara_estereo name="der" derecha="1.0"/>
+        <xacro:joint_camara_estereo name="der" izquierda="-1.0"/>
     </xacro:unless>
 </robot>
